File: kicad_source/HF50_FT81x_adapter.kicad_sch (KiCad schematic)
At the start: 6 parts, among them P1 LD09P33E4GX00LF, P2 KMDGX-8S-BS

Commit message: switched to THT parts
Parts:
- D1: footprint LEDs:LED_0603 -> LED_THT:LED_D3.0mm
- R1: footprint resistors:R_0603 -> Resistor_THT:R_Axial_DIN0207_L6.3mm_D2.5mm_P7.62mm_Horizontal
Changed lines of the file:
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@@
     (property "Reference" "R1" (id 0) (at 170.18 66.1416 90))
     (property "Value" "10k" (id 1) (at 170.18 68.453 90))
-    (property "Footprint" "resistors:R_0603" (id 2) (at 166.37 71.12 0)
+    (property "Footprint" "Resistor_THT:R_Axial_DIN0207_L6.3mm_D2.5mm_P7.62mm_Horizontal" (id 2) (at 166.37 71.12 0)
       (effects (font (size 1.27 1.27)) hide)
     )
@@
     (property "Reference" "D1" (id 0) (at 157.48 65.151 0))
     (property "Value" "150060GS75000" (id 1) (at 157.48 67.4624 0))
-    (property "Footprint" "LEDs:LED_0603" (id 2) (at 157.48 71.12 90)
+    (property "Footprint" "LED_THT:LED_D3.0mm" (id 2) (at 157.48 71.12 90)
       (effects (font (size 1.27 1.27)) hide)
     )
@@
     )
     (path "/00000000-0000-0000-0000-000060a6083a"
-      (reference "D1") (unit 1) (value "150060GS75000") (footprint "LEDs:LED_0603")
+      (reference "D1") (unit 1) (value "150060GS75000") (footprint "LED_THT:LED_D3.0mm")
     )
     (path "/00000000-0000-0000-0000-000060a6cf72"
@@
     )
     (path "/00000000-0000-0000-0000-000060a60105"
-      (reference "R1") (unit 1) (value "10k") (footprint "resistors:R_0603")
+      (reference "R1") (unit 1) (value "10k") (footprint "Resistor_THT:R_Axial_DIN0207_L6.3mm_D2.5mm_P7.62mm_Horizontal")
     )
   )
